File: psu_board/psu_board.sch (KiCad schematic (older format))
At the start: 27 parts, among them J1 Conn_02x08_Odd_Even, SW1 SW_SPST, U1 LM7812_TO220, U2 LM7805_TO220, U3 LM7912_TO220

Commit message: added fuse holder
Parts:
- removed J1: Conn_02x08_Odd_Even, Pin_Headers:Pin_Header_Straight_2x08_Pitch2.54mm, symbol Connector_Generic:Conn_02x08_Odd_Even
- removed SW1: SW_SPST, Microwave:ALIM, symbol Switch:SW_SPST
- added C2, C8: 4700uF, Capacitors_THT:CP_Radial_D18.0mm_P7.50mm, symbol Device:CP1
- added F1: Fuse, Fuse_Holders_and_Fuses:Fuseholder5x20_horiz_SemiClosed_Casing10x25mm, symbol Device:Fuse
- added J1: 12VAC_INPUT, digikey-footprints:spade_connector, symbol Connector:Conn_01x01_Male
- added J2: +5V, digikey-footprints:spade_connector, symbol Connector:Conn_01x01_Male
- added J3: +12V, digikey-footprints:spade_connector, symbol Connector:Conn_01x01_Male
- added J4: GND, digikey-footprints:spade_connector, symbol Connector:Conn_01x01_Male
- added J5: -12V, digikey-footprints:spade_connector, symbol Connector:Conn_01x01_Male
- added J6: GND_INPUT, digikey-footprints:spade_connector, symbol Connector:Conn_01x01_Male
- C1: value 10000uF -> 4700uF; footprint Capacitors_THT:CP_Radial_D22.0mm_P10.00mm_SnapIn -> Capacitors_THT:CP_Radial_D18.0mm_P7.50mm
- C7: renamed from C6; value 10000uF -> 4700uF; footprint Capacitors_THT:CP_Radial_D22.0mm_P10.00mm_SnapIn -> Capacitors_THT:CP_Radial_D18.0mm_P7.50mm
- renumbered C8 to C10, C2 to C3, C3 to C4, C4 to C5, C5 to C6, C7 to C9
Connections:
- wire segments 113 -> 116
- no-connect marks 4 -> 0
Other:
- moved on the sheet: D2, D9
